Commit message: fix(amr_description): 바퀴 충돌 원통을 얇게 해 제자리 회전 시 유효 바퀴 간격 오차 수정
Fortress(DART)가 원통-바닥 접촉점을 원통 안쪽 모서리에 잡아 유효 바퀴 간격이 0.34 → 0.298 m가 되고
odom이 회전을 12% 작게 쟀다. 충돌 원통을 폭 1 cm로 줄이고 반 폭 바깥으로 옮겨 0.341 m(오차 0.4%)로 맞춤.
보이는 바퀴(visual)는 그대로 폭 5 cm.

File: src/simulation/amr_description/urdf/properties.xacro (robot description, xacro)
@@ -15,4 +15,11 @@
   <xacro:property name="wheel_radius" value="0.1"/>
   <xacro:property name="wheel_width" value="0.05"/>
+  <!--
+    바퀴 충돌 원통 폭. 보이는 폭(wheel_width)과 따로 둔다.
+    Fortress(DART)는 원통-바닥 접촉점을 원통 안쪽 모서리에 잡아, 폭 5 cm 원통이면 제자리 회전에서
+    유효 바퀴 간격이 0.34 → 0.298 m로 줄어 odom이 회전을 12% 작게 잰다.
+    얇게 하고 폭의 절반만큼 바깥으로 옮겨 안쪽 모서리가 바퀴 중심선(wheel_separation / 2)에 오게 한다.
+  -->
+  <xacro:property name="wheel_contact_width" value="0.01"/>
   <xacro:property name="wheel_separation" value="0.34"/>
   <xacro:property name="wheel_mass" value="1.5"/>

File: src/simulation/amr_description/urdf/wheels.xacro (robot description, xacro)
@@ -15,8 +15,9 @@
         </material>
       </visual>
+      <!-- 충돌은 얇은 원통을 바깥으로 반 폭 옮겨 둔다 (properties.xacro wheel_contact_width 설명 참고) -->
       <collision>
-        <origin xyz="0 0 0" rpy="${pi/2} 0 0"/>
+        <origin xyz="0 ${reflect * wheel_contact_width / 2} 0" rpy="${pi/2} 0 0"/>
         <geometry>
-          <cylinder radius="${wheel_radius}" length="${wheel_width}"/>
+          <cylinder radius="${wheel_radius}" length="${wheel_contact_width}"/>
         </geometry>
       </collision>

Commit message: fix(amr_description): 바퀴 토크 한계 3 N·m·몸체 25 kg으로 확정 (#42 제동 거리 테스트)
- wheel_max_torque 속성 추가(20 → 3 N·m), base_mass 30 → 25 kg
- 일반 주행(가속 제한 ±1.0 m/s²)은 0/10/25 kg 모두 가속 1.05 s·제동 0.501 m로 명세 유지
- 가속 제한 없는 급정지 0.254/0.337/0.462 m로 #42 실험 모델과 같음 (20 N·m에서는 0.104/0.106 m로 질량 무관)
- README 주요 값 표가 #36 문단 때문에 끊겨 있던 것 수정

File: src/simulation/amr_description/urdf/properties.xacro (robot description, xacro)
@@ -9,5 +9,6 @@
   <xacro:property name="base_width" value="0.4"/>
   <xacro:property name="base_height" value="0.3"/>
-  <xacro:property name="base_mass" value="30.0"/>
+  <!-- 몸체 질량 [kg]. 제동 거리 테스트(#42) 권장: 소형 AGV 범위(Jackal 17 kg ~ RB-1 30 kg) 안의 25 kg -->
+  <xacro:property name="base_mass" value="25.0"/>
   <!-- 몸체 바닥과 지면 사이 간격 -->
   <xacro:property name="ground_clearance" value="0.03"/>
@@ -24,4 +25,10 @@
   <xacro:property name="wheel_separation" value="0.34"/>
   <xacro:property name="wheel_mass" value="1.5"/>
+  <!--
+    바퀴 조인트 최대 토크 [N·m]. 제동 거리 테스트(#42) 권장: 소형 AGV 허브모터 최대 토크 수준.
+    20 N·m면 모터가 한계에 닿지 않아 적재 질량이 가속·급정지에 거의 안 드러난다.
+    3 N·m × 2 / 0.1 m = 60 N → 최대 적재(25 kg, 전체 약 53.9 kg)에서도 1.1 m/s²로 명세 가속 1.0 m/s²를 낸다.
+  -->
+  <xacro:property name="wheel_max_torque" value="3.0"/>
   <!-- 캐스터: 앞뒤 2개, 마찰 없는 구 -->
   <xacro:property name="caster_radius" value="0.03"/>

File: src/simulation/amr_description/urdf/wheels.xacro (robot description, xacro)
@@ -36,5 +36,5 @@
       <origin xyz="0 ${reflect * wheel_separation / 2} ${wheel_radius - base_z}" rpy="0 0 0"/>
       <axis xyz="0 1 0"/>
-      <limit effort="20" velocity="${max_linear_velocity / wheel_radius}"/>
+      <limit effort="${wheel_max_torque}" velocity="${max_linear_velocity / wheel_radius}"/>
     </joint>
     <gazebo reference="${prefix}${side}_wheel_link">
