Commit message: feat(amr_gazebo): GT 주기 인자화와 사용 주의 사항 추가 (#25 리뷰 반영)
- gt_rate xacro·launch 인자 추가, 기본 50 → 100 Hz (민지·이진 요청)
- README: GT 속도는 이동 평균이 아니라 한 샘플(100Hz에서 10ms) 늦음을 실측 기록 (이진)
- README: world와 map 원점 차이, 지도 인계 시 매핑 시작 위치·방향 기록 규칙 (민지)

File: src/simulation/amr_description/urdf/amr.urdf.xacro (robot description, xacro)
@@ -2,5 +2,5 @@
 <!--
   AMR 조립 파일.
-    xacro amr.urdf.xacro namespace:=amr_01 payload_mass:=0.0
+    xacro amr.urdf.xacro namespace:=amr_01 payload_mass:=0.0 gt_rate:=100
   TF 트리 (docs/api.md 2장, prefix = "<namespace>/"):
     base_footprint
@@ -18,6 +18,9 @@
   <!-- 적재물 질량 [kg]. 몸체 질량에 더한다 -->
   <xacro:arg name="payload_mass" default="0.0"/>
+  <!-- GT 토픽 발행 주기 [Hz]. 평가용이라 실행마다 바꿀 수 있게 인자로 둔다 (제동 거리 테스트 등) -->
+  <xacro:arg name="gt_rate" default="100"/>
   <xacro:property name="namespace" value="$(arg namespace)"/>
   <xacro:property name="payload_mass" value="$(arg payload_mass)"/>
+  <xacro:property name="gt_rate" value="$(arg gt_rate)"/>
   <xacro:property name="prefix" value="${namespace + '/' if namespace else ''}"/>
   <xacro:property name="topic_ns" value="${'/' + namespace if namespace else ''}"/>

File: src/simulation/amr_description/urdf/gazebo.xacro (robot description, xacro)
@@ -44,5 +44,5 @@
       <tf_topic>${topic_ns}/ground_truth/tf</tf_topic>
       <dimensions>3</dimensions>
-      <odom_publish_frequency>50</odom_publish_frequency>
+      <odom_publish_frequency>${gt_rate}</odom_publish_frequency>
     </plugin>
   </gazebo>

Commit message: feat(amr_gazebo): enable_camera 인자로 RGBD 카메라 끄기
CPU 렌더링 sim에서 로봇 여러 대를 띄우면 카메라가 병목이라 끌 수 있게 한다 (#43 하연 리뷰).
- amr.urdf.xacro·sensors.xacro: enable_camera xacro 인자. false면 rgbd_camera 센서만 빼고 camera_link·광학 프레임 TF는 남긴다
- description·spawn_robot·sim launch: enable_camera 인자 (기본 true). false면 카메라 브리지·리매핑도 뺀다
- README·api.md 인자와 토픽 설명

File: src/simulation/amr_description/urdf/amr.urdf.xacro (robot description, xacro)
@@ -2,5 +2,5 @@
 <!--
   AMR 조립 파일.
-    xacro amr.urdf.xacro namespace:=amr_01 payload_mass:=0.0 gt_rate:=100
+    xacro amr.urdf.xacro namespace:=amr_01 payload_mass:=0.0 gt_rate:=100 enable_camera:=true
   TF 트리 (docs/api.md 2장, prefix = "<namespace>/"):
     base_footprint
@@ -20,7 +20,11 @@
   <!-- GT 토픽 발행 주기 [Hz]. 평가용이라 실행마다 바꿀 수 있게 인자로 둔다 (제동 거리 테스트 등) -->
   <xacro:arg name="gt_rate" default="100"/>
+  <!-- RGBD 카메라 센서를 만들지. false면 camera_link·광학 프레임(TF)은 남기고 Gazebo 센서만 뺀다.
+       CPU 렌더링 sim에서 로봇 여러 대를 띄울 때 카메라가 병목이라 끈다 (GCP 러너, #43 하연 리뷰) -->
+  <xacro:arg name="enable_camera" default="true"/>
   <xacro:property name="namespace" value="$(arg namespace)"/>
   <xacro:property name="payload_mass" value="$(arg payload_mass)"/>
   <xacro:property name="gt_rate" value="$(arg gt_rate)"/>
+  <xacro:property name="enable_camera" value="$(arg enable_camera)"/>
   <xacro:property name="prefix" value="${namespace + '/' if namespace else ''}"/>
   <xacro:property name="topic_ns" value="${'/' + namespace if namespace else ''}"/>

File: src/simulation/amr_description/urdf/sensors.xacro (robot description, xacro)
@@ -125,5 +125,7 @@
     RGB와 Depth를 한 센서로 낸다. 센서는 camera_link의 +x를 보고, 메시지 frame_id는 광학 프레임이다.
     Gazebo 토픽 camera/{image, depth_image, camera_info}는 spawn_robot.launch.py가 ROS 이름으로 바꾼다.
+    enable_camera가 false면 센서를 만들지 않는다 (링크·TF는 위에서 그대로 만든다).
   -->
+  <xacro:if value="${enable_camera}">
   <gazebo reference="${prefix}camera_link">
     <sensor name="rgbd_camera" type="rgbd_camera">
@@ -158,4 +160,5 @@
     </sensor>
   </gazebo>
+  </xacro:if>
   <gazebo reference="${prefix}imu_link">
     <sensor name="imu" type="imu">

Commit message: feat(amr_detection): YOLO 학습 데이터 수집 노드(collect_dataset)와 라벨 카메라(label_camera), 모델 라벨, 화물 상자별 모델

File: src/simulation/amr_description/urdf/amr.urdf.xacro (robot description, xacro)
@@ -2,5 +2,5 @@
 <!--
   AMR 조립 파일.
-    xacro amr.urdf.xacro namespace:=amr_01 payload_mass:=0.0 gt_rate:=100 enable_camera:=true
+    xacro amr.urdf.xacro namespace:=amr_01 payload_mass:=0.0 gt_rate:=100 enable_camera:=true label_camera:=false
   TF 트리 (docs/api.md 2장, prefix = "<namespace>/"):
     base_footprint
@@ -23,8 +23,12 @@
        CPU 렌더링 sim에서 로봇 여러 대를 띄울 때 카메라가 병목이라 끈다 (GCP 러너, #43 하연 리뷰) -->
   <xacro:arg name="enable_camera" default="true"/>
+  <!-- 라벨 카메라(YOLO 학습 데이터 수집 전용). RGBD 카메라와 같은 자리·화각에서 라벨 붙은 물체의 화면 속 상자를 낸다.
+       렌더링 부담이 있어 기본으로 끈다 (experiments/yolo) -->
+  <xacro:arg name="label_camera" default="false"/>
   <xacro:property name="namespace" value="$(arg namespace)"/>
   <xacro:property name="payload_mass" value="$(arg payload_mass)"/>
   <xacro:property name="gt_rate" value="$(arg gt_rate)"/>
   <xacro:property name="enable_camera" value="$(arg enable_camera)"/>
+  <xacro:property name="label_camera" value="$(arg label_camera)"/>
   <xacro:property name="prefix" value="${namespace + '/' if namespace else ''}"/>
   <xacro:property name="topic_ns" value="${'/' + namespace if namespace else ''}"/>

File: src/simulation/amr_description/urdf/sensors.xacro (robot description, xacro)
@@ -161,4 +161,32 @@
   </gazebo>
   </xacro:if>
+  <!--
+    라벨 카메라 (YOLO 학습 데이터 수집 전용, label_camera:=true). RGBD 카메라와 같은 링크·화각·해상도라
+    같은 시각의 RGB 영상과 픽셀이 맞는다. Label 플러그인이 붙은 모델마다 화면에 보이는 부분의 2D 상자를 낸다
+    (가려진 부분은 빼고, 모델 단위로 하나). ROS: /<ns>/camera/labels (vision_msgs/Detection2DArray)
+  -->
+  <xacro:if value="${label_camera}">
+  <gazebo reference="${prefix}camera_link">
+    <sensor name="label_camera" type="boundingbox_camera">
+      <always_on>true</always_on>
+      <visualize>false</visualize>
+      <update_rate>10</update_rate>
+      <topic>${topic_ns}/camera/labels</topic>
+      <ignition_frame_id>${prefix}camera_optical_frame</ignition_frame_id>
+      <camera>
+        <box_type>2d</box_type>
+        <horizontal_fov>${radians(rgbd['horizontal_fov'])}</horizontal_fov>
+        <image>
+          <width>${rgbd['width']}</width>
+          <height>${rgbd['height']}</height>
+        </image>
+        <clip>
+          <near>${rgbd['range_min']}</near>
+          <far>${rgbd['range_max']}</far>
+        </clip>
+      </camera>
+    </sensor>
+  </gazebo>
+  </xacro:if>
   <gazebo reference="${prefix}imu_link">
     <sensor name="imu" type="imu">

Commit message: feat(amr_gazebo): 연구 2 RL Gazebo 평가 환경 (2D와 같은 시나리오·지표, 적재 질량 토크 한계)
- worlds/rl_eval.sdf, launch/rl_eval.launch.py: 빈 월드 + 로봇(payload_mass) + 에피소드 노드
- amr_description: xacro 인자 max_linear_acceleration (기본 1.0). 평가 환경은 10으로 풀어 바퀴 토크 한계가 질량에 따라 가감속을 정함 (#55)
- rl_eval.py: research2 dynamics·scenarios를 그대로 읽어 같은 시드 → 같은 시나리오, 가속 구간, 통로 벽·돌발 장애물, 2D와 같은 지표(EpisodeTracker)
- rl_eval_node.py: 에피소드 실행, 장애물은 trigger_x 통과 순간 움직임, 벽은 지나감(충돌 비트마스크)
- rl_policies.py: 시험 정책 cruise·brake, 외부 정책 모듈:함수
- experiments/rl_gazebo_eval: 같은 정책 2D 실행·비교, 60쌍 중 57쌍 결과 일치 (S2 30/30)
- 테스트 16개 (2D 시나리오 일치, 배치, 판정, 정책)

File: src/simulation/amr_description/urdf/amr.urdf.xacro (robot description, xacro)
@@ -23,4 +23,7 @@
        CPU 렌더링 sim에서 로봇 여러 대를 띄울 때 카메라가 병목이라 끈다 (GCP 러너, #43 하연 리뷰) -->
   <xacro:arg name="enable_camera" default="true"/>
+  <!-- DiffDrive 선가속 상한 [m/s²]. 기본 1.0(명세). 바퀴 토크 한계(3 N·m)가 적재 질량에 따라 가감속을 정하게
+       하려면 크게 준다 (연구 2 RL 평가 환경 rl_eval.launch.py, #55 이진 제동 실험: 1.0이면 질량과 상관없이 같다) -->
+  <xacro:arg name="max_linear_acceleration" default="1.0"/>
   <xacro:property name="namespace" value="$(arg namespace)"/>
   <xacro:property name="payload_mass" value="$(arg payload_mass)"/>

File: src/simulation/amr_description/urdf/properties.xacro (robot description, xacro)
@@ -37,5 +37,5 @@
   <!-- 동역학 제한 (명세: 최대 속도 2.0 m/s, 가속도 1.0 m/s², 회전 1.5 rad/s) -->
   <xacro:property name="max_linear_velocity" value="2.0"/>
-  <xacro:property name="max_linear_acceleration" value="1.0"/>
+  <xacro:property name="max_linear_acceleration" value="$(arg max_linear_acceleration)"/>
   <xacro:property name="max_angular_velocity" value="1.5"/>
   <!-- 명세에 없는 임시값. Nav2 DWB acc_lim_theta(amr_bringup/config/nav2_params.yaml)와 맞춘다 -->
